File: pico.kicad_pcb (KiCad board)
At the start: 2 copper layers, 103 x 101.2 mm, 89 parts, among them J101 Programming, J102 ???, J103 XT60, J104 MR30, J105 MR30, Q101 IRFS7434TRL7PP, Q102 SQJ142EP-T1_GE3, Q103 SQJ142EP-T1_GE3, Q104 SQJ142EP-T1_GE3, Q105 SQJ142EP-T1_GE3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

Commit message: seprate motors
Parts:
- removed C134: 47u, Capacitor_THT:CP_Radial_D6.3mm_P2.50mm
- removed C135, C139, C144, C145, C146, C155, C156, C160, C165, C166: 1u, COMPONENTS:1206_Resistor
- removed C136, C138, C147, C159: 100n, COMPONENTS:1206_Resistor
- removed C137, C150: 47n, COMPONENTS:1206_Resistor
- removed C140, C141, C151, C152, C161, C162: 47u low ESR, Capacitor_THT:CP_Radial_D6.3mm_P2.50mm
- removed C142, C143, C153, C154, C163, C164: 10u, COMPONENTS:1206_Resistor
- removed J104, J105: MR30, Connector_AMASS:AMASS_MR30PW-FB_1x03_P3.50mm_Horizontal
- removed JP101, JP102, JP103, JP104, JP105, JP106: SolderJumper_3_Open, Jumper:SolderJumper-3_P1.3mm_Open_RoundedPad1.0x1.5mm_NumberLabels
- removed Q102, Q103, Q104, Q105, Q106, Q107, Q108, Q109, Q110, Q111, Q112, Q113: SQJ142EP-T1_GE3, JLCPCB_Transistors_Thyristors:POWERPAK-SO-8_L5.9-W4.9-P1.27-BL
- removed R106, R111: 100k, COMPONENTS:1206_Resistor
- removed R107, R108, R109, R110, R112, R113: 2m, COMPONENTS:1206_Resistor
- removed U104: DRV8323SRTAT, JLCPCB_Power_Supply_Chip:WQFN-40_L6.0-W6.0-P0.50-TL-EP4.5
- added C201: 47u, Capacitor_THT:CP_Radial_D6.3mm_P2.50mm, F.Cu at (153.0, 53.5)
- added C202: 1u, COMPONENTS:1206_Resistor, F.Cu at (147.2, 51.2)
- added C203: 100n, COMPONENTS:1206_Resistor, F.Cu at (147.2, 54.5)
- added C204: 47n, COMPONENTS:1206_Resistor, F.Cu at (55.0, 77.2)
- added C205: 100n, COMPONENTS:1206_Resistor, F.Cu at (59.0, 90.2)
- added C206: 1u, COMPONENTS:1206_Resistor, F.Cu at (62.1, 83.8)
- added C207: 47u low ESR, Capacitor_THT:CP_Radial_D6.3mm_P2.50mm, F.Cu at (31.3, 66.1)
- added C208: 10u, COMPONENTS:1206_Resistor, F.Cu at (26.4, 70.8)
- added C209: 1u, COMPONENTS:1206_Resistor, F.Cu at (26.4, 68.5)
- added C210: 47u low ESR, Capacitor_THT:CP_Radial_D6.3mm_P2.50mm, F.Cu at (44.3, 89.7)
- added C211: 10u, COMPONENTS:1206_Resistor, F.Cu at (42.0, 88.5)
- added C212: 1u, COMPONENTS:1206_Resistor, F.Cu at (39.8, 88.5)
- added C213: 47u low ESR, Capacitor_THT:CP_Radial_D6.3mm_P2.50mm, F.Cu at (44.2, 95.1)
- added C214: 10u, COMPONENTS:1206_Resistor, F.Cu at (42.0, 96.5)
- added C215: 1u, COMPONENTS:1206_Resistor, F.Cu at (39.8, 96.5)
- added J201: MR30, Connector_AMASS:AMASS_MR30PW-FB_1x03_P3.50mm_Horizontal, F.Cu at (17.3, 78.0)
- added JP201: SolderJumper_3_Open, Jumper:SolderJumper-3_P1.3mm_Open_RoundedPad1.0x1.5mm_NumberLabels, F.Cu at (45.8, 77.1)
- added JP202: SolderJumper_3_Open, Jumper:SolderJumper-3_P1.3mm_Open_RoundedPad1.0x1.5mm_NumberLabels, F.Cu at (47.5, 83.5)
- added JP203: SolderJumper_3_Open, Jumper:SolderJumper-3_P1.3mm_Open_RoundedPad1.0x1.5mm_NumberLabels, F.Cu at (25.7, 100.9)
- added Q201: SQJ142EP-T1_GE3, JLCPCB_Transistors_Thyristors:POWERPAK-SO-8_L5.9-W4.9-P1.27-BL, F.Cu at (20.7, 70.0)
- added Q202: SQJ142EP-T1_GE3, JLCPCB_Transistors_Thyristors:POWERPAK-SO-8_L5.9-W4.9-P1.27-BL, F.Cu at (23.9, 76.5)
- added Q203: SQJ142EP-T1_GE3, JLCPCB_Transistors_Thyristors:POWERPAK-SO-8_L5.9-W4.9-P1.27-BL, F.Cu at (27.0, 88.5)
- added Q204: SQJ142EP-T1_GE3, JLCPCB_Transistors_Thyristors:POWERPAK-SO-8_L5.9-W4.9-P1.27-BL, F.Cu at (23.9, 81.5)
- added Q205: SQJ142EP-T1_GE3, JLCPCB_Transistors_Thyristors:POWERPAK-SO-8_L5.9-W4.9-P1.27-BL, F.Cu at (27.0, 93.8)
- added Q206: SQJ142EP-T1_GE3, JLCPCB_Transistors_Thyristors:POWERPAK-SO-8_L5.9-W4.9-P1.27-BL, F.Cu at (20.5, 93.5)
- added R201: 100k, COMPONENTS:1206_Resistor, F.Cu at (55.4, 91.4)
- added R202: 2m, COMPONENTS:1206_Resistor, F.Cu at (31.0, 77.1)
- added R203: 2m, COMPONENTS:1206_Resistor, F.Cu at (31.0, 82.1)
- added R204: 2m, COMPONENTS:1206_Resistor, F.Cu at (20.5, 100.8)
- added U201: DRV8323SRTAT, JLCPCB_Power_Supply_Chip:WQFN-40_L6.0-W6.0-P0.50-TL-EP4.5, F.Cu at (54.0, 84.8)
- moved J102 165.2 mm to (200.1, 125.1)
- moved C113 152.1 mm to (200.8, 121.2)
- moved C103 149.8 mm to (204.8, 126.1)
- moved C110 145.8 mm to (200.8, 117.9)
- moved C131 144.4 mm to (206.7, 117.9)
- moved C104 143.3 mm to (188.1, 110.3)
- moved C105 143.3 mm to (188.1, 118.2)
- moved C132 140.4 mm to (206.7, 121.2)
- moved C129 135.3 mm to (188.1, 126.0)
- moved R104 114.3 mm to (212.7, 111.3)
- moved R105 114.3 mm to (212.7, 114.6)
- moved C107 106.0 mm to (200.8, 114.6)
- moved C101 101.8 mm to (200.8, 108.0)
- moved C102 100.4 mm to (200.8, 111.3)
- moved C118 100.4 mm to (206.7, 111.3)
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Routing:
- net A_Z: track 47.4 -> 0.00 mm
- net /MotorDriver/Z: track 0.00 -> 47.4 mm
- net A_Z_S_H: track 43.2 -> 0.00 mm
- net /MotorDriver/Z_S_H: track 0.00 -> 43.2 mm
- net A_Z_L: track 40.2 -> 0.00 mm
- net /MotorDriver/Z_L: track 0.00 -> 40.2 mm
- net A_Z_S_L: track 37.5 -> 0.00 mm
- net /MotorDriver/Z_S_L: track 0.00 -> 37.5 mm
- net A_Z_H: track 37.0 -> 0.00 mm
- net /MotorDriver/Z_H: track 0.00 -> 37.0 mm
- net A_X_H: track 36.1 -> 0.00 mm
- net /MotorDriver/X_H: track 0.00 -> 36.1 mm
- net A_X: track 35.9 -> 0.00 mm
- net /MotorDriver/X: track 0.00 -> 35.9 mm
- net A_Y: track 34.0 -> 0.00 mm
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- added copper zone on F.Cu, net (none)
- added copper zone on F.Cu, net /MotorDriver/Y
- added copper zone on F.Cu, net /MotorDriver/Z
- added copper zone on F.Cu, net /MotorDriver/Z_S_H
- removed copper zone on F.Cu, net A_X_S_H
- removed copper zone on F.Cu, net A_Y
- removed copper zone on F.Cu, net A_Y_S_H
- removed copper zone on F.Cu, net A_Z
- removed copper zone on F.Cu, net A_Z_S_H

Commit message: finished driverA
Parts:
- moved C201 99.4 mm to (55.0, 70.2), turned to 135 degrees
- moved C203 98.8 mm to (50.2, 73.0), turned to 135 degrees
- moved C202 95.8 mm to (54.0, 73.2), turned to 135 degrees
- moved C204 1.59 mm to (56.5, 76.6)
Routing:
- net +BATT: track 36.0 -> 82.2 mm, vias 0 -> 9
- net Net-(U201-VCP): track 0.00 -> 8.75 mm
- net Net-(U201-CPH): track 4.18 -> 5.95 mm
- net Net-(U201-CPL): track 5.47 -> 6.72 mm
- added copper zone on F.Cu, net /MotorDriver/X
- added copper zone on F.Cu, net /MotorDriver/X_S_H
- added copper zone on F.Cu, net /MotorDriver/Y_S_H
- removed copper zone on F.Cu, net (none)
