File: MotorDriver.kicad_sch (KiCad schematic)
At the start: 30 parts, among them J201 MR30, Q201 SQJ142EP-T1_GE3, Q202 SQJ142EP-T1_GE3, Q203 SQJ142EP-T1_GE3, Q204 SQJ142EP-T1_GE3, Q205 SQJ142EP-T1_GE3, Q206 SQJ142EP-T1_GE3, U201 DRV8323SRTAT

Commit message: finished driverA
Changed lines of the file:
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@@
+	(wire
+		(pts
+			(xy 103.505 97.79) (xy 106.68 97.79)
+		)
+		(stroke
+			(width 0)
+			(type default)
+		)
+	)
 	(wire
 		(pts
@@
 	(hierarchical_label "+BATT"
 		(shape input)
-		(at 106.68 97.79 180)
-		(effects
-			(font
+		(at 103.505 97.79 180)
+		(effects
+			(font

Commit message: why every commit needs a message
Changed lines of the file:
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@@
 	(text "DRIVER_CHANNEL_CONNECTION\n"
 		(exclude_from_sim no)
-		(at 115.316 116.078 90)
+		(at 115.57 115.57 90)
 		(effects
 			(font

Commit message: Good progress
Parts:
- removed J201: MR30, Connector_AMASS:AMASS_MR30PW-FB_1x03_P3.50mm_Horizontal, symbol Connector_Generic:Conn_01x03
- added H201, H202, H203: MountingHole_Pad, Connector_Wire:SolderWire-2sqmm_1x01_D2mm_OD3.9mm, symbol Mechanical:MountingHole_Pad
Connections:
- net X: now also H201.1
- net Y: now also H202.1
- net Z: now also H203.1

Commit message: via stiching trzeba
Changed lines of the file:
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@@
 	(wire
 		(pts
-			(xy 103.505 97.79) (xy 106.68 97.79)
+			(xy 85.09 115.57) (xy 96.52 115.57)
 		)
 		(stroke
@@
 	(wire
 		(pts
+			(xy 96.52 115.57) (xy 96.52 97.79)
+		)
+		(stroke
+			(width 0)
+			(type default)
+		)
+	)
+	(wire
+		(pts
 			(xy 91.44 66.04) (xy 91.44 64.77)
 		)
@@
 		(pts
 			(xy 80.01 95.25) (xy 76.2 95.25)
+		)
+		(stroke
+			(width 0)
+			(type default)
+		)
+	)
+	(wire
+		(pts
+			(xy 96.52 97.79) (xy 106.68 97.79)
 		)
 		(stroke
@@
 	(hierarchical_label "+BATT"
 		(shape input)
-		(at 103.505 97.79 180)
-		(effects
-			(font
+		(at 85.09 115.57 180)
+		(effects
+			(font

Commit message: m, mn,
Parts:
- R202, R203, R204: footprint COMPONENTS:1206_Resistor -> Resistor_SMD:R_2512_6332Metric_Pad1.40x3.35mm_HandSolder
Changed lines of the file:
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@@
 			)
 		)
-		(property "Footprint" "COMPONENTS:1206_Resistor"
+		(property "Footprint" "Resistor_SMD:R_2512_6332Metric_Pad1.40x3.35mm_HandSolder"
 			(at 203.962 60.96 90)
 			(effects
@@
 			)
 		)
-		(property "Footprint" "COMPONENTS:1206_Resistor"
+		(property "Footprint" "Resistor_SMD:R_2512_6332Metric_Pad1.40x3.35mm_HandSolder"
 			(at 89.662 60.96 90)
 			(effects
@@
 			)
 		)
-		(property "Footprint" "COMPONENTS:1206_Resistor"
+		(property "Footprint" "Resistor_SMD:R_2512_6332Metric_Pad1.40x3.35mm_HandSolder"
 			(at 146.812 60.96 90)
 			(effects
